File: Schematic/AudioAmplifierPCB.kicad_sch (KiCad schematic)
At the start: 14 parts, among them J1 Screw_Terminal_01x02, J2 AudioJack2_Ground, J3 AudioJack2_Ground, U1 LM7812_TO220, U2 NE5534

Commit message: designing pcb
Parts:
- removed R2: 24K, symbol Device:R_Variable
- added D1: LED, LED_SMD:LED_0805_2012Metric_Pad1.15x1.40mm_HandSolder, symbol Device:LED
- added R2: 1k, Resistor_SMD:R_0805_2012Metric_Pad1.20x1.40mm_HandSolder, symbol Device:R_Small
- added RV1: 10k, Potentiometer_THT:Potentiometer_Piher_PT-10-H05_Horizontal, symbol Device:R_Potentiometer_Trim_US
- C1, C2, C4: footprint (none) -> Capacitor_THT:CP_Radial_D4.0mm_P1.50mm
- C3, C5: footprint (none) -> Capacitor_SMD:C_0805_2012Metric_Pad1.18x1.45mm_HandSolder
- C6: footprint (none) -> Capacitor_THT:C_Disc_D3.0mm_W1.6mm_P2.50mm
- J1: footprint (none) -> TerminalBlock:TerminalBlock_MaiXu_MX126-5.0-02P_1x02_P5.00mm
- J2, J3: footprint (none) -> Connector_Audio:Jack_3.5mm_CUI_SJ-3523-SMT_Horizontal
- R1, R4: footprint (none) -> Resistor_SMD:R_0805_2012Metric_Pad1.20x1.40mm_HandSolder
- U2: footprint (none) -> Package_TO_SOT_THT:TO-220-3_Vertical
Connections:
- net +12V: now also R2.1
- net GND: now also D1.1 (K), RV1.3
- net at C3.1, R1.1, U2.2 (-): now also RV1.1
- net at C3.2, C4.2, C6.2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: now also RV1.2
- new net: D1.2 (A), R2.2
